Commit message: A sucessfull creation of a rig with the lidar and oakd using xacro and being modular

File: ros_ws/src/seeker_sim/model/Rigs/Rig_simpelBox/model.sdf.xacro (robot description, xacro)
@@ -1,10 +1,9 @@
 <?xml version="1.0" ?>
-<robot xmlns:xacro="http://www.ros.org/wiki/xacro"> <!-- tag name doesn't matter for SDF output -->
-  <!-- Parameters -->
+  <sdf version="1.10" xmlns:xacro="http://www.ros.org/wiki/xacro">
+      <!-- Parameters -->
   <xacro:property name="box_size_x" value="0.6"/>
   <xacro:property name="box_size_y" value="0.4"/>
-  <xacro:property name="box_size_z" value="0.5"/>   <!-- change me -->
-  <sdf version="1.10">
-    <model name="Rig_simpelBox">
+  <xacro:property name="box_size_z" value="0.5"/>
+    <xacro:macro name="Rig_simpelBox">
     <pose>0 0 0 0 0 0</pose>
     <static>false</static>
@@ -18,5 +17,4 @@
       </visual>
     </link>
-  </model>
+  </xacro:macro>
   </sdf>
-</robot>
