Commit message: made the husky into a xacro file and attateched the rig to it

File: ros_ws/src/seeker_sim/model/Rigs/Rig_simpelBox_xacro/model.sdf.xacro (robot description, xacro)
@@ -5,7 +5,8 @@
   <xacro:property name="box_size_y" value="0.4"/>
   <xacro:property name="box_size_z" value="0.5"/>
-    <xacro:macro name="Rig_simpelBox_xacro">
+    <xacro:macro name="Rig_simpelBox_xacro" params='offset:="0 0 0 0 0 0" UGV_link'>
     <static>false</static>
     <link name="box_link">
+      <pose>${offset}</pose>
       <gravity>true</gravity>
       <collision name="c">
