Commit message: Fixed RSP and bridged the oakd to Rviz

File: ros_ws/src/seeker_sim/model/Assemblies/Rig5/model.sdf.xacro (robot description, xacro)
@@ -6,5 +6,5 @@
   <xacro:include filename="$(find seeker_sim)/model/UGV/Husky_stripped_xacro/model.sdf.xacro"/>
   <model name="Rig4" canonical_link='UGV_link'>
-    <xacro:property name="oakd_x_offset" value="${0*cm2m}"/>
+    <xacro:property name="oakd_x_offset" value="${4*cm2m}"/>
     <xacro:property name="oakd_y_offset" value="${0*cm2m}"/>
     <xacro:property name="oakd_z_offset" value="${0*cm2m}"/>
@@ -27,8 +27,8 @@
     <!-- <origin xyz="${oakd_x_offset} ${oakd_y_offset} ${oakd_z_offset}"/> -->
     <link name="rig_bottom_link">
-    <pose relative_to="rig_link">0 0 ${-0.5*box_size_z} 0 ${pi/2} 0</pose>
+    <pose relative_to="rig_link">0 0 ${-0.5*box_size_z} 0 0 0</pose>
     </link>
     <link name="rig_top_link">
-    <pose relative_to="rig_link">0 0 ${0.5*box_size_z} 0 ${-pi/2} 0</pose>
+    <pose relative_to="rig_link">0 0 ${0.5*box_size_z} 0 0 0</pose>
     </link>
     <link name="rig_front_link">
@@ -36,14 +36,14 @@
     </link>
     <link name="rig_back_link">
-    <pose relative_to="rig_link">${-0.5*box_size_x} 0 0 0 0 ${pi}</pose>
+    <pose relative_to="rig_link">${-0.5*box_size_x} 0 0 0 0 0</pose>
     </link>
     <link name="rig_left_link">
-    <pose relative_to="rig_link">0 ${0.5*box_size_y} 0 0 0 ${pi/2}</pose>
+    <pose relative_to="rig_link">0 ${0.5*box_size_y} 0 0 0 0</pose>
     </link>
     <link name="rig_right_link">
-    <pose relative_to="rig_link">0 ${-0.5*box_size_y} 0 0 0 ${-pi/2}</pose>
+    <pose relative_to="rig_link">0 ${-0.5*box_size_y} 0 0 0 0</pose>
     </link>
-    <xacro:oakd parent_link="rig_left_link" xyz="${oakd_x_offset} ${oakd_y_offset} ${oakd_z_offset}" rpy="0 0 0"/>
-    <xacro:mid360_lidar parent_link="rig_top_link" xyz="${mid360_lidar_x_offset} ${mid360_lidar_x_offset} ${mid360_lidar_x_offset}" rpy="0 ${pi/2} 0"/>
+    <xacro:oakd parent_link="rig_front_link" xyz="${oakd_x_offset} ${oakd_y_offset} ${oakd_z_offset}" rpy="0 0 0"/>
+    <xacro:mid360_lidar parent_link="rig_top_link" xyz="${mid360_lidar_x_offset} ${mid360_lidar_y_offset} ${mid360_lidar_z_offset}" rpy="0 0 0"/>
     <xacro:Husky_stripped_xacro base_link="UGV_link"/>
     <joint name="base_joint" type="fixed">

File: ros_ws/src/seeker_sim/model/Sensors/mid360_lidar/model.sdf.xacro (robot description, xacro)
@@ -1,5 +1,5 @@
 <?xml version="1.0" ?>
 <sdf version="1.10" xmlns:xacro="http://ros.org/wiki/xacro">
-  <xacro:macro name="mid360_lidar" params='name:="mid360_lidar" parent_link xyz:="0 0 0" rpy:="0 0 0"'>
+  <xacro:macro name="mid360_lidar" params='name:=mid360_lidar parent_link xyz:="0 0 0" rpy:="0 0 0"'>
     <xacro:property name="base_frame" value="${name}_link"/>
       <link name="${base_frame}">
@@ -96,5 +96,5 @@
                   </noise>
                 </lidar>
-                <topic>/lidar/mid360/points</topic>  <!-- Gazebo Transport topic -->
+                <topic>/lidar_points</topic>  <!-- Gazebo Transport topic -->
                 <pose relative_to="${base_frame}">0 0 0 0 0 0</pose>
           </sensor>

File: ros_ws/src/seeker_sim/model/Sensors/oakd/model.sdf.xacro (robot description, xacro)
@@ -2,5 +2,5 @@
 <sdf version="1.11" xmlns:xacro="http://ros.org/wiki/xacro">
   <xacro:include filename="$(find seeker_sim)/model/Sensors/oakd/common.sdf.xacro" />
-    <xacro:macro name="oakd" params='name:="oakd_pro" parent_link xyz:="0 0 0" rpy:="0 0 0"'>
+    <xacro:macro name="oakd" params='name:=oakd_pro parent_link xyz:="0 0 0" rpy:="0 0 0"'>
       <xacro:property name="mass"       value="0.061"/>
       <xacro:property name="baseline"   value="0.075" />
@@ -24,5 +24,5 @@
         </visual>
         <collision name="${base_frame}_collision">
-          <pose>${collision_offset_x} ${collision_offset_y} ${collision_offset_z} 0 0 0</pose>
+          <pose relative_to="${base_frame}">${collision_offset_x} ${collision_offset_y} ${collision_offset_z} 0 0 0</pose>
           <geometry>
             <box>
@@ -45,4 +45,5 @@
       <!-- RGB Camera -->
       <link name="${name}_rgb_camera_frame">
+        <pose relative_to="${base_frame}">0 0 0 0 0 0</pose>
         <xacro:inertial_dummy/>
         <sensor name="${name}_rgbd_sensor" type="rgbd_camera">
@@ -77,5 +78,5 @@
         <parent>${base_frame}</parent>
         <child>${name}_rgb_camera_frame</child>
-        <pose>0 0 0 0 0 0</pose>
+        <pose relative_to="${base_frame}">0 0 0 0 0 0</pose>
       </joint>
       <link name="${name}_rgb_camera_optical_frame">
@@ -83,5 +84,5 @@
       </link>
       <joint name="${name}_rgb_camera_optical_joint" type="fixed">
-        <pose>0 0 0 -${M_PI/2} 0.0 -${M_PI/2}</pose>
+        <pose relative_to="${base_frame}">0 0 0 0.0 0.0 0.0</pose>
         <parent>${name}_rgb_camera_frame</parent>
         <child>${name}_rgb_camera_optical_frame</child>
@@ -91,5 +92,5 @@
         <parent>${name}_rgb_camera_optical_frame</parent>
         <child>${name}_rgb_camera_sensor_mount</child>
-        <pose>0 0 0 0 0 0</pose>
+        <pose relative_to="${base_frame}">0 0 0 0 0 0</pose>
       </joint>
       <!-- Left Camera -->
@@ -118,5 +119,5 @@
         <parent>${base_frame}</parent>
         <child>${name}_left_camera_frame</child>
-        <pose>0 ${baseline/2} 0 0 0 0</pose>
+        <pose relative_to="${base_frame}">0 ${baseline/2} 0 0 0 0</pose>
       </joint>
       <link name="${name}_left_camera_optical_frame">
@@ -124,5 +125,5 @@
       </link>
       <joint name="${name}_left_camera_optical_joint" type="fixed">
-        <pose>0 0 0 -${M_PI/2} 0.0 -${M_PI/2}</pose>
+        <pose relative_to="${base_frame}">0 0 0 -${M_PI/2} 0.0 -${M_PI/2}</pose>
         <parent>${name}_left_camera_frame</parent>
         <child>${name}_left_camera_optical_frame</child>
@@ -153,5 +154,5 @@
         <parent>${base_frame}</parent>
         <child>${name}_right_camera_frame</child>
-        <pose>0 -${baseline/2} 0 0 0 0</pose>
+        <pose relative_to="${base_frame}">0 -${baseline/2} 0 0 0 0</pose>
       </joint>
       <link name="${name}_right_camera_optical_frame">
@@ -159,5 +160,5 @@
       </link>
       <joint name="${name}_right_camera_optical_joint" type="fixed">
-        <pose>0 0 0 -${M_PI/2} 0.0 -${M_PI/2}</pose>
+        <pose relative_to="${base_frame}">0 0 0 -${M_PI/2} 0.0 -${M_PI/2}</pose>
         <parent>${name}_right_camera_frame</parent>
         <child>${name}_right_camera_optical_frame</child>
@@ -199,5 +200,5 @@
         <parent>${base_frame}</parent>
         <child>${name}_imu_frame</child>
-        <pose>0 0 0 -${M_PI/2} 0 -${M_PI/2}</pose>
+        <pose relative_to="${base_frame}">0 0 0 -${M_PI/2} 0 -${M_PI/2}</pose>
       </joint>
       <joint name="oakd_mount" type="fixed">

File: ros_ws/src/seeker_sim/model/UGV/Husky_stripped_xacro/model.sdf.xacro (robot description, xacro)
@@ -431,8 +431,8 @@
       <wheel_radius>0.165</wheel_radius>
       <!-- Topics / frames -->
-      <topic>/model/husky/cmd_vel</topic>
-      <odom_topic>/model/husky/odometry</odom_topic>
+      <topic>/cmd_vel</topic>
+      <odom_topic>/odometry</odom_topic>
       <odom_frame>odom</odom_frame>
-      <robot_base_frame>base_link</robot_base_frame>
+      <robot_base_frame>${base_link}</robot_base_frame>
       <publish_odom>true</publish_odom>
       <publish_tf>false</publish_tf>
