Commit message: initial navigation commit

File: ros_ws/src/hs_description/sdf/hs.sdf.xacro (robot description, xacro)
@@ -1,5 +1,5 @@
 <?xml version="1.0" ?>
 <sdf version="1.11" xmlns:xacro="http://ros.org/wiki/xacro">
-  <xacro:include filename="$(find hs_description)/urdf/oakd.sdf.xacro" />
+  <xacro:include filename="$(find hs_description)/sdf/oakd.sdf.xacro" />
   <model name="heavy_seeker" canonical_link='base_link'>
     <link name="base_link">

File: ros_ws/src/hs_description/sdf/oakd.sdf.xacro (robot description, xacro)
@@ -1,6 +1,6 @@
 <?xml version="1.0"?>
 <sdf version="1.11" xmlns:xacro="http://ros.org/wiki/xacro">
-  <xacro:include filename="$(find hs_description)/urdf/common.sdf.xacro" />
-    <xacro:macro name="oakd" params="name:=oakd_pro parent_link *origin">
+  <xacro:include filename="$(find hs_description)/sdf/common.sdf.xacro" />
+    <xacro:macro name="oakd" params="name:=oakd parent_link *origin">
       <xacro:property name="mass"       value="0.061"/>
       <xacro:property name="baseline"   value="0.075" />
@@ -204,5 +204,5 @@
         <parent>${base_frame}</parent>
         <child>${name}_imu_frame</child>
-        <pose>0 0 0 -${M_PI/2} 0 -${M_PI/2}</pose>
+        <pose>0 0 0 -0.5 0.5 -0.5 0.5</pose>
       </joint>
     </xacro:macro>

Commit message: add lidar imu to ekf

File: ros_ws/src/hs_description/sdf/hs.sdf.xacro (robot description, xacro)
@@ -8,12 +8,12 @@
     </link>
     <!-- Mechanical properties -->
-    <xacro:property name="oakd_x_offset" value="${0*cm2m}"/>
-    <xacro:property name="oakd_y_offset" value="${0*cm2m}"/>
-    <xacro:property name="oakd_z_offset" value="${0*cm2m}"/>
+    <xacro:property name="oakd_x_offset" value="${15*cm2m}"/>
+    <xacro:property name="oakd_y_offset" value="${15*cm2m}"/>
+    <xacro:property name="oakd_z_offset" value="${15*cm2m}"/>
     <!-- Sensor definitions -->
-    <!-- <xacro:oakd parent_link="base_link"> -->
+    <xacro:oakd parent_link="base_link">
       <!-- <origin xyz="${oakd_x_offset} ${oakd_y_offset} ${oakd_z_offset}"/> -->
-      <!-- <pose>${oakd_x_offset} ${oakd_y_offset} ${oakd_z_offset} 0 0 0</pose> -->
-    <!-- </xacro:oakd> -->
+      <pose>${oakd_x_offset} ${oakd_y_offset} ${oakd_z_offset} 0 0 0</pose>
+    </xacro:oakd>
     <xacro:mid360_lidar parent_link="base_link" xyz="0 0 0" rpy="0 0 0"/>
     <link name="base_footprint">

File: ros_ws/src/hs_description/sdf/livox.sdf.xacro (robot description, xacro)
@@ -104,4 +104,11 @@
         <child>${base_frame}</child>
       </joint>
+      <link name="livox_frame">
+        <pose relative_to="${base_frame}">0 0 0 0 0 0</pose>
+      </link>
+      <joint name="livox_frame_joint" type="fixed">
+        <parent>${base_frame}</parent>
+        <child>livox_frame</child>
+      </joint>
   </xacro:macro>
 </sdf>

File: ros_ws/src/hs_description/sdf/oakd.sdf.xacro (robot description, xacro)
@@ -205,9 +205,9 @@
         <child>${name}_imu_frame</child>
         <!-- From oakd description file. Rotation is mirrored around all axes -->
-        <!-- <pose>-0.008 -0.037945 -0.00079 ${M_PI} ${M_PI/2.0} 0.0</pose> -->
+        <pose>-0.008 -0.037945 -0.00079 ${M_PI} ${M_PI/2.0} 0.0</pose>
         <!-- rotation around z-axis is mirrored -->
         <!-- <pose>0 0 0 0.0 ${M_PI/2} 0.0</pose> -->
         <!-- rotation around x-axis is mirrored -->
-        <pose>0 0 0 0.0 -${M_PI/2} 0.0</pose>
+        <!-- <pose>0 0 0 0.0 -${M_PI/2} 0.0</pose> -->
         <!-- rotation around y-axis mirrored -->
         <!-- <pose>0 0 0 ${M_PI/2} -${M_PI/2} ${M_PI/2}</pose> -->
