Commit message: Bringup of waypoint nav w navsat. Work done together by Josef, Matthias, Vlad and Christopher

File: ros_ws/src/hs_description/sdf/oakd.sdf.xacro (robot description, xacro)
@@ -204,5 +204,5 @@
         <parent>${base_frame}</parent>
         <child>${name}_imu_frame</child>
-        <pose>0 0 0 -0.5 0.5 -0.5 0.5</pose>
+        <pose rotation_format="quat_xyzw">0 0 0 -0.5 0.5 -0.5 0.5</pose>
       </joint>
     </xacro:macro>

File: ros_ws/src/seeker_sim/model/Assemblies/Rig5/model.sdf.xacro (robot description, xacro)
@@ -5,4 +5,5 @@
   <xacro:include filename="$(find seeker_sim)/model/Sensors/mid360_lidar/model.sdf.xacro"/>
   <xacro:include filename="$(find seeker_sim)/model/UGV/Husky_stripped_xacro/model.sdf.xacro"/>
+  <xacro:include filename="$(find seeker_sim)/model/Sensors/navsat_gnss/model.sdf.xacro"/>
   <model name="Rig5" canonical_link='UGV_link'>
     <xacro:property name="oakd_x_offset" value="${4*cm2m}"/>
@@ -13,4 +14,7 @@
     <xacro:property name="mid360_lidar_z_offset" value="${0*cm2m}"/>
     <xacro:property name="rig_pos_relative_2_UGV" value="0 0 0.45 0 0 0"/>
+    <xacro:property name="gnss_x_offset" value="${0*cm2m}"/>
+    <xacro:property name="gnss_y_offset" value="${0*cm2m}"/>
+    <xacro:property name="gnss_z_offset" value="${15*cm2m}"/>
     <link name="rig_link">
       <inertial>
@@ -44,4 +48,5 @@
     <pose relative_to="rig_link">0 ${-0.5*box_size_y} 0 0 0 0</pose>
     </link>
+    <xacro:navsat_gnss parent_link="rig_top_link" xyz="${gnss_x_offset} ${gnss_y_offset} ${gnss_z_offset}" rpy="0 0 0"/>
     <xacro:oakd parent_link="rig_front_link" xyz="${oakd_x_offset} ${oakd_y_offset} ${oakd_z_offset}" rpy="0 0 0"/>
     <xacro:mid360_lidar parent_link="rig_top_link" xyz="${mid360_lidar_x_offset} ${mid360_lidar_y_offset} ${mid360_lidar_z_offset}" rpy="0 0 0"/>

File: ros_ws/src/seeker_sim/model/Sensors/navsat_gnss/model.sdf.xacro (robot description, xacro)
@@ -12,4 +12,5 @@
       </inertial>
       <sensor name="gnss" type="navsat">
+        <topic>/gps/fix</topic>
         <always_on>true</always_on>
         <update_rate>10</update_rate>
@@ -25,5 +26,6 @@
         </navsat>
         <plugin name="gz::sim::systems::NavSat" filename="gz-sim-navsat-system">
-          <topic>/gps/fix</topic>
+          <!-- <topic>/gps/fix</topic>
+          <frame_id>gnss_link</frame_id> -->
         </plugin>
       </sensor>

File: ros_ws/src/seeker_sim/model/UGV/Husky_stripped_xacro/model.sdf.xacro (robot description, xacro)
@@ -125,4 +125,25 @@
       </visual>
     </link>
+    <link name="base_footprint">
+      <visual name="base_footprint_visual">
+        <geometry>
+          <box>
+            <size>0.80 0.5709 0.095</size>
+          </box>
+        </geometry>
+        <material>
+          <ambient>0.1 0.1 0.1 1.0</ambient>
+          <diffuse>0.0 0.6 0.8 1.0</diffuse>
+          <specular>0.2 0.2 0.2 1.0</specular>
+          <emissive>0 0 0 1.0</emissive>
+        </material>
+        <transparency>0.65</transparency>
+      </visual>
+    </link>
+  <joint name="base_footprint_to_base_link" type="fixed">
+    <parent>${base_link}</parent>
+    <child>base_footprint</child>
+    <pose relative_to="${base_link}">0 0 0.046 0 0 0</pose>
+  </joint>
     <link name="front_left_wheel_link">
       <pose frame="">0.256 0.2854 0.03282 0 -0 0</pose>
@@ -432,6 +453,8 @@
       <!-- Topics / frames -->
       <topic>/cmd_vel</topic>
-      <odom_topic>/odometry</odom_topic>
+      <odom_topic>/odometry/wheel</odom_topic>
       <odom_frame>odom</odom_frame>
+      <frame_id>odom</frame_id>
+      <child_frame_id>${base_link}</child_frame_id>
       <robot_base_frame>${base_link}</robot_base_frame>
       <publish_odom>true</publish_odom>
