Commit message: move `.sdf` model files to hs_description
- Move files that can be used independently of simulation
- Modify hs_description launch file to publish `tf2` from new files
- Modify `seeker_sim.launch.py` to use hs_description instead of its custom launch file

File: ros_ws/src/hs_description/model/Assemblies/Rig2/model.sdf.xacro (robot description, xacro)
@@ -1,7 +1,6 @@
 <?xml version="1.0" ?>
 <sdf version="1.10" xmlns:xacro="http://www.ros.org/wiki/xacro">
-  <xacro:include filename="$(find seeker_sim)/model/Rigs/Rig_simpelBox_xacro/model.sdf.xacro" />
-  <xacro:include filename="$(find seeker_sim)/model/Sensors/oakd/model.sdf.xacro"/>
-  <xacro:include filename="$(find seeker_sim)/model/Sensors/mid360_lidar/model.sdf.xacro"/>
+  <xacro:include filename="$(find hs_description)/model/Rigs/Rig_simpelBox_xacro/model.sdf.xacro" />
+  <xacro:include filename="$(find hs_description)/model/Sensors/oakd/model.sdf.xacro"/>
   <model name="Rig2" canonical_link='rig_link'>
     <link name="rig_link">
@@ -11,8 +10,5 @@
     <xacro:property name="oakd_y_offset" value="${0*cm2m}"/>
     <xacro:property name="oakd_z_offset" value="${0*cm2m}"/>
-    <xacro:property name="mid360_lidar_x_offset" value="${0*cm2m}"/>
-    <xacro:property name="mid360_lidar_y_offset" value="${0*cm2m}"/>
-    <xacro:property name="mid360_lidar_z_offset" value="${0*cm2m}"/>
-    <xacro:Rig_simpelBox_xacro/>
+    <xacro:Rig_simpelBox_xacro offset="0 0 0 0 0 0" UGV_link="rig_link"/>
     <!--use box_size_x,box_size_y,box_size_z in the offset to allign sensor placement-->
     <!-- <origin xyz="${oakd_x_offset} ${oakd_y_offset} ${oakd_z_offset}"/> -->
@@ -36,34 +32,27 @@
     </link>
     <xacro:oakd parent_link="rig_left_link" xyz="${oakd_x_offset} ${oakd_y_offset} ${oakd_z_offset}" rpy="0 0 0"/>
-    <xacro:mid360_lidar parent_link="rig_top_link" xyz="${mid360_lidar_x_offset} ${mid360_lidar_x_offset} ${mid360_lidar_x_offset}" rpy="0 ${pi/2} 0"/>
     <joint name="base_joint" type="fixed">
       <parent>rig_link</parent>
       <child>rig_bottom_link</child>
-      <!-- ingen pose behövs här -->
     </joint>
     <joint name="top_joint" type="fixed">
       <parent>rig_link</parent>
       <child>rig_top_link</child>
-      <!-- ingen pose behövs här -->
     </joint>
     <joint name="right_side_joint" type="fixed">
       <parent>rig_link</parent>
       <child>rig_right_link</child>
-      <!-- ingen pose behövs här -->
     </joint>
     <joint name="left_side_joint" type="fixed">
       <parent>rig_link</parent>
       <child>rig_left_link</child>
-      <!-- ingen pose behövs här -->
     </joint>
     <joint name="left_front_joint" type="fixed">
       <parent>rig_link</parent>
       <child>rig_front_link</child>
-      <!-- ingen pose behövs här -->
     </joint>
     <joint name="left_back_joint" type="fixed">
       <parent>rig_link</parent>
       <child>rig_back_link</child>
-      <!-- ingen pose behövs här -->
     </joint>
     <joint name="box_mount" type="fixed">

File: ros_ws/src/hs_description/model/Assemblies/Rig3/model.sdf.xacro (robot description, xacro)
@@ -1,9 +1,11 @@
 <?xml version="1.0" ?>
 <sdf version="1.10" xmlns:xacro="http://www.ros.org/wiki/xacro">
-  <xacro:include filename="$(find seeker_sim)/model/Rigs/Rig_simpelBox_xacro/model.sdf.xacro" />
-  <xacro:include filename="$(find seeker_sim)/model/Sensors/oakd/model.sdf.xacro"/>
-  <xacro:include filename="$(find seeker_sim)/model/Sensors/mid360_lidar/model.sdf.xacro"/>
-  <xacro:include filename="$(find seeker_sim)/model/UGV/Husky_stripped_xacro/model.sdf.xacro"/>
-  <model name="Rig4" canonical_link='UGV_link'>
+  <xacro:include filename="$(find hs_description)/model/Rigs/Rig_simpelBox_xacro/model.sdf.xacro" />
+  <xacro:include filename="$(find hs_description)/model/Sensors/oakd/model.sdf.xacro"/>
+  <xacro:include filename="$(find hs_description)/model/Sensors/mid360_lidar/model.sdf.xacro"/>
+  <model name="Rig2" canonical_link='rig_link'>
+    <link name="rig_link">
+      <must_be_base_link>false</must_be_base_link>
+    </link>
     <xacro:property name="oakd_x_offset" value="${0*cm2m}"/>
     <xacro:property name="oakd_y_offset" value="${0*cm2m}"/>
@@ -12,16 +14,5 @@
     <xacro:property name="mid360_lidar_y_offset" value="${0*cm2m}"/>
     <xacro:property name="mid360_lidar_z_offset" value="${0*cm2m}"/>
-    <xacro:property name="rig_pos_relative_2_UGV" value="0 0 0.45 0 0 0"/>
-    <link name="rig_link">
-      <inertial>
-      <mass>0.1</mass>
-      <inertia>
-        <ixx>0.001</ixx><iyy>0.001</iyy><izz>0.001</izz>
-        <ixy>0</ixy><ixz>0</ixz><iyz>0</iyz>
-      </inertia>
-      </inertial>
-      <pose relative_to="UGV_link">${rig_pos_relative_2_UGV}</pose>
-    </link>
-    <xacro:Rig_simpelBox_xacro UGV_link="UGV_link" offset="${rig_pos_relative_2_UGV}"/>
+    <xacro:Rig_simpelBox_xacro/>
     <!--use box_size_x,box_size_y,box_size_z in the offset to allign sensor placement-->
     <!-- <origin xyz="${oakd_x_offset} ${oakd_y_offset} ${oakd_z_offset}"/> -->
@@ -46,34 +37,27 @@
     <xacro:oakd parent_link="rig_left_link" xyz="${oakd_x_offset} ${oakd_y_offset} ${oakd_z_offset}" rpy="0 0 0"/>
     <xacro:mid360_lidar parent_link="rig_top_link" xyz="${mid360_lidar_x_offset} ${mid360_lidar_x_offset} ${mid360_lidar_x_offset}" rpy="0 ${pi/2} 0"/>
-    <xacro:Husky_stripped_xacro base_link="UGV_link"/>
     <joint name="base_joint" type="fixed">
       <parent>rig_link</parent>
       <child>rig_bottom_link</child>
-      <!-- ingen pose behövs här -->
     </joint>
     <joint name="top_joint" type="fixed">
       <parent>rig_link</parent>
       <child>rig_top_link</child>
-      <!-- ingen pose behövs här -->
     </joint>
     <joint name="right_side_joint" type="fixed">
       <parent>rig_link</parent>
       <child>rig_right_link</child>
-      <!-- ingen pose behövs här -->
     </joint>
     <joint name="left_side_joint" type="fixed">
       <parent>rig_link</parent>
       <child>rig_left_link</child>
-      <!-- ingen pose behövs här -->
     </joint>
     <joint name="left_front_joint" type="fixed">
       <parent>rig_link</parent>
       <child>rig_front_link</child>
-      <!-- ingen pose behövs här -->
     </joint>
     <joint name="left_back_joint" type="fixed">
       <parent>rig_link</parent>
       <child>rig_back_link</child>
-      <!-- ingen pose behövs här -->
     </joint>
     <joint name="box_mount" type="fixed">
@@ -81,8 +65,4 @@
       <child>box_link</child>
     </joint>
-    <joint name="UGV_rig_mount" type="fixed">
-      <parent>UGV_link</parent>
-      <child>rig_link</child>
-    </joint>
     <pose>0 0 0 0 0 0</pose>
   </model>

File: ros_ws/src/hs_description/model/Assemblies/Rig4/model.sdf.xacro (robot description, xacro)
@@ -1,14 +1,27 @@
 <?xml version="1.0" ?>
 <sdf version="1.10" xmlns:xacro="http://www.ros.org/wiki/xacro">
-  <xacro:include filename="$(find seeker_sim)/model/Rigs/Rig_simpelBox_xacro/model.sdf.xacro" />
-  <xacro:include filename="$(find seeker_sim)/model/Sensors/oakd/model.sdf.xacro"/>
-  <model name="Rig2" canonical_link='rig_link'>
-    <link name="rig_link">
-      <must_be_base_link>false</must_be_base_link>
-    </link>
+  <xacro:include filename="$(find hs_description)/model/Rigs/Rig_simpelBox_xacro/model.sdf.xacro" />
+  <xacro:include filename="$(find hs_description)/model/Sensors/oakd/model.sdf.xacro"/>
+  <xacro:include filename="$(find hs_description)/model/Sensors/mid360_lidar/model.sdf.xacro"/>
+  <xacro:include filename="$(find hs_description)/model/UGV/Husky_stripped_xacro/model.sdf.xacro"/>
+  <model name="Rig4" canonical_link='UGV_link'>
     <xacro:property name="oakd_x_offset" value="${0*cm2m}"/>
     <xacro:property name="oakd_y_offset" value="${0*cm2m}"/>
     <xacro:property name="oakd_z_offset" value="${0*cm2m}"/>
-    <xacro:Rig_simpelBox_xacro offset="0 0 0 0 0 0" UGV_link="rig_link"/>
+    <xacro:property name="mid360_lidar_x_offset" value="${0*cm2m}"/>
+    <xacro:property name="mid360_lidar_y_offset" value="${0*cm2m}"/>
+    <xacro:property name="mid360_lidar_z_offset" value="${0*cm2m}"/>
+    <xacro:property name="rig_pos_relative_2_UGV" value="0 0 0.45 0 0 0"/>
+    <link name="rig_link">
+      <inertial>
+      <mass>0.1</mass>
+      <inertia>
+        <ixx>0.001</ixx><iyy>0.001</iyy><izz>0.001</izz>
+        <ixy>0</ixy><ixz>0</ixz><iyz>0</iyz>
+      </inertia>
+      </inertial>
+      <pose relative_to="UGV_link">${rig_pos_relative_2_UGV}</pose>
+    </link>
+    <xacro:Rig_simpelBox_xacro UGV_link="UGV_link" offset="${rig_pos_relative_2_UGV}"/>
     <!--use box_size_x,box_size_y,box_size_z in the offset to allign sensor placement-->
     <!-- <origin xyz="${oakd_x_offset} ${oakd_y_offset} ${oakd_z_offset}"/> -->
@@ -32,33 +45,29 @@
     </link>
     <xacro:oakd parent_link="rig_left_link" xyz="${oakd_x_offset} ${oakd_y_offset} ${oakd_z_offset}" rpy="0 0 0"/>
+    <xacro:mid360_lidar parent_link="rig_top_link" xyz="${mid360_lidar_x_offset} ${mid360_lidar_x_offset} ${mid360_lidar_x_offset}" rpy="0 ${pi/2} 0"/>
+    <xacro:Husky_stripped_xacro base_link="UGV_link"/>
     <joint name="base_joint" type="fixed">
       <parent>rig_link</parent>
       <child>rig_bottom_link</child>
-      <!-- ingen pose behövs här -->
     </joint>
     <joint name="top_joint" type="fixed">
       <parent>rig_link</parent>
       <child>rig_top_link</child>
-      <!-- ingen pose behövs här -->
     </joint>
     <joint name="right_side_joint" type="fixed">
       <parent>rig_link</parent>
       <child>rig_right_link</child>
-      <!-- ingen pose behövs här -->
     </joint>
     <joint name="left_side_joint" type="fixed">
       <parent>rig_link</parent>
       <child>rig_left_link</child>
-      <!-- ingen pose behövs här -->
     </joint>
     <joint name="left_front_joint" type="fixed">
       <parent>rig_link</parent>
       <child>rig_front_link</child>
-      <!-- ingen pose behövs här -->
     </joint>
     <joint name="left_back_joint" type="fixed">
       <parent>rig_link</parent>
       <child>rig_back_link</child>
-      <!-- ingen pose behövs här -->
     </joint>
     <joint name="box_mount" type="fixed">
@@ -66,4 +75,8 @@
       <child>box_link</child>
     </joint>
+    <joint name="UGV_rig_mount" type="fixed">
+      <parent>UGV_link</parent>
+      <child>rig_link</child>
+    </joint>
     <pose>0 0 0 0 0 0</pose>
   </model>

File: ros_ws/src/hs_description/model/Assemblies/Rig5/model.sdf.xacro (robot description, xacro)
@@ -1,9 +1,9 @@
 <?xml version="1.0" ?>
 <sdf version="1.10" xmlns:xacro="http://www.ros.org/wiki/xacro">
-  <xacro:include filename="$(find seeker_sim)/model/Rigs/Rig_simpelBox_xacro/model.sdf.xacro" />
-  <xacro:include filename="$(find seeker_sim)/model/Sensors/oakd/model.sdf.xacro"/>
-  <xacro:include filename="$(find seeker_sim)/model/Sensors/mid360_lidar/model.sdf.xacro"/>
-  <xacro:include filename="$(find seeker_sim)/model/UGV/Husky_stripped_xacro/model.sdf.xacro"/>
-  <xacro:include filename="$(find seeker_sim)/model/Sensors/navsat_gnss/model.sdf.xacro"/>
+  <xacro:include filename="$(find hs_description)/model/Rigs/Rig_simpelBox_xacro/model.sdf.xacro" />
+  <xacro:include filename="$(find hs_description)/model/Sensors/oakd/model.sdf.xacro"/>
+  <xacro:include filename="$(find hs_description)/model/Sensors/mid360_lidar/model.sdf.xacro"/>
+  <xacro:include filename="$(find hs_description)/model/UGV/Husky_stripped_xacro/model.sdf.xacro"/>
+  <xacro:include filename="$(find hs_description)/model/Sensors/navsat_gnss/model.sdf.xacro"/>
   <model name="Rig5" canonical_link='UGV_link'>
     <xacro:property name="oakd_x_offset" value="${4*cm2m}"/>
@@ -55,30 +55,24 @@
       <parent>rig_link</parent>
       <child>rig_bottom_link</child>
-      <!-- ingen pose behövs här -->
     </joint>
     <joint name="top_joint" type="fixed">
       <parent>rig_link</parent>
       <child>rig_top_link</child>
-      <!-- ingen pose behövs här -->
     </joint>
     <joint name="right_side_joint" type="fixed">
       <parent>rig_link</parent>
       <child>rig_right_link</child>
-      <!-- ingen pose behövs här -->
     </joint>
     <joint name="left_side_joint" type="fixed">
       <parent>rig_link</parent>
       <child>rig_left_link</child>
-      <!-- ingen pose behövs här -->
     </joint>
     <joint name="left_front_joint" type="fixed">
       <parent>rig_link</parent>
       <child>rig_front_link</child>
-      <!-- ingen pose behövs här -->
     </joint>
     <joint name="left_back_joint" type="fixed">
       <parent>rig_link</parent>
       <child>rig_back_link</child>
-      <!-- ingen pose behövs här -->
     </joint>
     <joint name="box_mount" type="fixed">

File: ros_ws/src/hs_description/model/Sensors/navsat_gnss/model.sdf.xacro (robot description, xacro)
@@ -2,5 +2,4 @@
 <sdf version="1.10" xmlns:xacro="http://www.ros.org/wiki/xacro">
   <xacro:macro name="navsat_gnss" params="parent_link xyz rpy name:='gnss' rate:='10'">
-    <!-- Länk som bär sensorn -->
     <link name="${name}_link">
       <inertial>
@@ -26,10 +25,7 @@
         </navsat>
         <plugin name="gz::sim::systems::NavSat" filename="gz-sim-navsat-system">
-          <!-- <topic>/gps/fix</topic>
-          <frame_id>gnss_link</frame_id> -->
         </plugin>
       </sensor>
     </link>
-    <!-- Fäst länken på vår rigg/UGV -->
     <joint name="${name}_mount" type="fixed">
       <parent>${parent_link}</parent>

File: ros_ws/src/hs_description/model/Sensors/oakd/model.sdf.xacro (robot description, xacro)
@@ -1,5 +1,5 @@
 <?xml version="1.0"?>
 <sdf version="1.11" xmlns:xacro="http://ros.org/wiki/xacro">
-  <xacro:include filename="$(find seeker_sim)/model/Sensors/oakd/common.sdf.xacro" />
+  <xacro:include filename="$(find hs_description)/model/Sensors/oakd/common.sdf.xacro" />
     <xacro:macro name="oakd" params='name:=oakd_pro parent_link xyz:="0 0 0" rpy:="0 0 0"'>
       <xacro:property name="mass"       value="0.061"/>
