Commit message: change gnss_frame

File: ros_ws/src/hs_description/model/Sensors/navsat_gnss/model.sdf.xacro (robot description, xacro)
@@ -2,5 +2,5 @@
 <sdf version="1.10" xmlns:xacro="http://www.ros.org/wiki/xacro">
   <xacro:macro name="navsat_gnss" params="parent_link xyz rpy name:='gnss' rate:='10'">
-    <link name="${name}_link">
+    <link name="${name}_frame">
       <inertial>
         <mass>0.01</mass>
@@ -30,5 +30,5 @@
     <joint name="${name}_mount" type="fixed">
       <parent>${parent_link}</parent>
-      <child>${name}_link</child>
+      <child>${name}_frame</child>
       <pose>${xyz} ${rpy}</pose>
     </joint>
