Commit message: add Rig6
- this `.sdf` should reflect actual husky build

File: ros_ws/src/hs_description/model/Rigs/Rig_simpelBox_xacro/model.sdf.xacro (robot description, xacro)
@@ -1,18 +1,13 @@
 <?xml version="1.0" ?>
   <sdf version="1.10" xmlns:xacro="http://www.ros.org/wiki/xacro">
-      <!-- Parameters -->
-  <xacro:property name="box_size_x" value="0.6"/>
-  <xacro:property name="box_size_y" value="0.4"/>
-  <xacro:property name="box_size_z" value="0.5"/>
-    <xacro:macro name="Rig_simpelBox_xacro" params='offset:="0 0 0 0 0 0" UGV_link'>
+    <xacro:macro name="Rig_simpelBox_xacro" params='size:="0.6 0.4 0.5" offset:="0 0 0 0 0 0"'>
     <static>false</static>
     <link name="box_link">
-      <pose>${offset}</pose>
       <gravity>true</gravity>
       <collision name="c">
-        <geometry><box><size>${box_size_x} ${box_size_y} ${box_size_z}</size></box></geometry>
+        <geometry><box><size>${size}</size></box></geometry>
       </collision>
       <visual name="v">
-        <geometry><box><size>${box_size_x} ${box_size_y} ${box_size_z}</size></box></geometry>
+        <geometry><box><size>${size}</size></box></geometry>
       </visual>
     </link>

File: ros_ws/src/hs_description/model/Sensors/mid360_lidar/model.sdf.xacro (robot description, xacro)
@@ -2,5 +2,5 @@
 <sdf version="1.10" xmlns:xacro="http://ros.org/wiki/xacro">
   <xacro:macro name="mid360_lidar" params='name:=mid360_lidar parent_link xyz:="0 0 0" rpy:="0 0 0"'>
-    <xacro:property name="base_frame" value="${name}_link"/>
+    <xacro:property name="base_frame" value="livox_frame"/>
       <link name="${base_frame}">
         <pose relative_to="${parent_link}">${xyz} ${rpy}</pose>
@@ -97,5 +97,4 @@
                 </lidar>
                 <topic>/lidar_points</topic>  <!-- Gazebo Transport topic -->
-                <pose relative_to="${base_frame}">0 0 0 0 0 0</pose>
           </sensor>
       </link>

File: ros_ws/src/hs_description/model/Sensors/navsat_gnss/model.sdf.xacro (robot description, xacro)
@@ -31,5 +31,5 @@
       <parent>${parent_link}</parent>
       <child>${name}_link</child>
-      <pose>${xyz} ${rpy}</pose>
+      <pose relative_to="${parent_link}">${xyz} ${rpy}</pose>
     </joint>
   </xacro:macro>

File: ros_ws/src/hs_description/model/UGV/Husky_stripped_xacro/model.sdf.xacro (robot description, xacro)
@@ -434,10 +434,10 @@
       </axis>
     </joint>
-    <link name="Top_plate_link">
-    </link>
-    <joint name="Top_plate_joint" type="fixed">
-      <child>Top_plate_link</child>
+    <link name="top_plate_link">
+      <pose relative_to ="${base_link}">0.0812 0 0.245 0 -0 0</pose>
+    </link>
+    <joint name="top_plate_joint" type="fixed">
+      <child>top_plate_link</child>
       <parent>${base_link}</parent>
-      <pose relative_to ="${base_link}">0.0812 0 0.245 0 -0 0</pose>
     </joint>
     <static>false</static>
