Commit message: fixed the frame positions of the real light seeker model

File: ros_ws/src/s_description/model/UGV/Light_seeker/model.sdf.xacro (robot description, xacro)
@@ -2,6 +2,7 @@
 <sdf version="1.6" xmlns:xacro="http://www.ros.org/wiki/xacro">
   <xacro:macro name="Light_seeker" params='base_link:="base_link"'>
+    <xacro:property name="groundz_z_offset" value="${0.1}"/>
     <link name="${base_link}">
-      <pose frame="">0 0 0.0 0 -0 0</pose>
+      <pose frame="">0 0 0 0 0 0</pose>
       <inertial>
         <pose frame="">0 0 0.062329 0 -0 0</pose>
@@ -33,11 +34,12 @@
       <velocity_decay/>
     <link name="base_footprint">
-      <pose frame="">0 0 ${-0.165+0.03282} 0 0 0</pose>
+      <pose frame="">0 0 -0.33 0 0 0</pose>
       <visual name="base_footprint_visual">
+        <pose frame="">0 0 0 0 0 0</pose>
         <geometry>
           <box>
             <!-- pos: 0.256 -0.2854 wheel: 0.1143-->
             <!--<size>${(0.2854+0.1143)*2} ${0.256*2} 0.01</size>-->
-            <size>0.88 ${0.44+0.1146*2} 0.01</size>
+            <size>0.94 ${0.345*2 + 0.145} 0.01</size>
           </box>
         </geometry>
@@ -54,8 +56,8 @@
     <parent>${base_link}</parent>
     <child>base_footprint</child>
-    <pose relative_to="${base_link}">0 0 0.046 0 0 0</pose>
+    <pose relative_to="${base_link}">0 0 -0.33 0 0 0</pose> <!--0.046? why?-->
   </joint>
     <link name="front_left_wheel_link">
-      <pose frame="">0.256 0.2854 0.03282 0 -0 0</pose>
+      <pose frame="">0.295 0.345 -0.155 0 -0 0</pose>
       <inertial>
         <pose frame="">0 0 0 0 -0 0</pose>
@@ -71,9 +73,9 @@
       </inertial>
       <collision name="front_left_wheel_link_collision">
-        <pose frame="">0 0 0 1.5707963267948966 -0 0</pose>
-        <geometry>
-          <cylinder>
-            <length>0.1143</length>
-            <radius>0.1651</radius>
+        <pose frame="">0 0 0 0 ${pi/2} ${pi/2}</pose>
+        <geometry>
+          <cylinder>
+            <length>0.145</length>
+            <radius>0.175</radius>
           </cylinder>
         </geometry>
@@ -97,10 +99,14 @@
       </collision>
       <visual name="front_left_wheel_link_visual">
-        <pose frame="">0 0 0 0 -0 0</pose>
-        <geometry>
-          <mesh>
+        <pose frame="">0 0 0 0 ${pi/2} ${pi/2}</pose>
+        <geometry>
+          <cylinder>
+            <length>0.145</length>
+            <radius>0.175</radius>
+          </cylinder>
+          <!--<mesh>
             <scale>1 1 1</scale>
             <uri>model://Husky_stripped_xacro/meshes/wheel.dae</uri>
-          </mesh>
+          </mesh>-->
         </geometry>
       </visual>
@@ -129,7 +135,7 @@
     </joint>
     <link name="front_right_wheel_link">
-      <pose frame="">0.256 -0.2854 0.03282 0 -0 0</pose>
-      <inertial>
-        <pose frame="">0 0 0 0 -0 0</pose>
+      <pose frame="">0.295 -0.345 -0.155 0 -0 0</pose>
+      <inertial>
+        <pose frame="">0 0 0 0 0 0</pose>
         <mass>2.637</mass>
         <inertia>
@@ -143,9 +149,9 @@
       </inertial>
       <collision name="front_right_wheel_link_collision">
-        <pose frame="">0 0 0 1.5707963267948966 -0 0</pose>
-        <geometry>
-          <cylinder>
-            <length>0.1143</length>
-            <radius>0.1651</radius>
+      <pose frame="">0 0 0 0 ${pi/2} ${pi/2}</pose>
+        <geometry>
+          <cylinder>
+            <length>0.145</length>
+            <radius>0.175</radius>
           </cylinder>
         </geometry>
@@ -169,10 +175,14 @@
       </collision>
       <visual name="front_right_wheel_link_visual">
-        <pose frame="">0 0 0 0 -0 0</pose>
-        <geometry>
-          <mesh>
+          <pose frame="">0 0 0 0 ${pi/2} ${pi/2}</pose>
+        <geometry>
+          <cylinder>
+            <length>0.145</length>
+            <radius>0.175</radius>
+          </cylinder>
+          <!--<mesh>
             <scale>1 1 1</scale>
             <uri>model://Husky_stripped_xacro/meshes/wheel.dae</uri>
-          </mesh>
+          </mesh>-->
         </geometry>
       </visual>
@@ -201,7 +211,7 @@
     </joint>
     <link name="rear_left_wheel_link">
-      <pose frame="">-0.256 0.2854 0.03282 0 -0 0</pose>
-      <inertial>
-        <pose frame="">0 0 0 0 -0 0</pose>
+      <pose frame="">-0.295 0.345 -0.155 0 -0 0</pose>
+      <inertial>
+        <pose frame="">0 0 0 0 0 0</pose>
         <mass>2.637</mass>
         <inertia>
@@ -215,9 +225,9 @@
       </inertial>
       <collision name="rear_left_wheel_link_collision">
-        <pose frame="">0 0 0 1.5707963267948966 -0 0</pose>
-        <geometry>
-          <cylinder>
-            <length>0.1143</length>
-            <radius>0.1651</radius>
+        <pose frame="">0 0 0 0 ${pi/2} ${pi/2}</pose>
+        <geometry>
+          <cylinder>
+            <length>0.145</length>
+            <radius>0.175</radius>
           </cylinder>
         </geometry>
@@ -241,10 +251,14 @@
       </collision>
       <visual name="rear_left_wheel_link_visual">
-        <pose frame="">0 0 0 0 -0 0</pose>
-        <geometry>
-          <mesh>
+        <pose frame="">0 0 0 0 ${pi/2} ${pi/2}</pose>
+        <geometry>
+          <cylinder>
+            <length>0.145</length>
+            <radius>0.175</radius>
+          </cylinder>
+          <!--<mesh>
             <scale>1 1 1</scale>
             <uri>model://Husky_stripped_xacro/meshes/wheel.dae</uri>
-          </mesh>
+          </mesh>-->
         </geometry>
       </visual>
@@ -273,7 +287,7 @@
     </joint>
     <link name="rear_right_wheel_link">
-      <pose frame="">-0.256 -0.2854 0.03282 0 -0 0</pose>
-      <inertial>
-        <pose frame="">0 0 0 0 -0 0</pose>
+      <pose frame="">-0.295 -0.345 -0.155 0 -0 0</pose>
+      <inertial>
+        <pose frame="">0 0 0 0 0 0</pose>
         <mass>2.637</mass>
         <inertia>
@@ -287,9 +301,9 @@
       </inertial>
       <collision name="rear_right_wheel_link_collision">
-        <pose frame="">0 0 0 1.5707963267948966 -0 0</pose>
-        <geometry>
-          <cylinder>
-            <length>0.1143</length>
-            <radius>0.1651</radius>
+        <pose frame="">0 0 0 0 ${pi/2} ${pi/2}</pose>
+        <geometry>
+          <cylinder>
+            <length>0.145</length>
+            <radius>0.175</radius>
           </cylinder>
         </geometry>
@@ -313,10 +327,14 @@
       </collision>
       <visual name="rear_right_wheel_link_visual">
-        <pose frame="">0 0 0 0 -0 0</pose>
-        <geometry>
-          <mesh>
+        <pose frame="">0 0 0 0 ${pi/2} ${pi/2}</pose>
+        <geometry>
+          <cylinder>
+            <length>0.145</length>
+            <radius>0.175</radius>
+          </cylinder>
+          <!--<mesh>
             <scale>1 1 1</scale>
             <uri>model://Husky_stripped_xacro/meshes/wheel.dae</uri>
-          </mesh>
+          </mesh>-->
         </geometry>
       </visual>
@@ -349,5 +367,5 @@
       <child>Top_plate_link</child>
       <parent>${base_link}</parent>
-      <pose relative_to ="${base_link}">0.0812 0 0.245 0 -0 0</pose>
+      <pose relative_to ="${base_link}">0 0 0.095 0 0 0</pose>
     </joint>
     <static>false</static>
@@ -359,6 +377,6 @@
       <right_joint>rear_right_wheel_joint</right_joint>
       <!-- Tune to your model’s geometry -->
-      <wheel_separation>0.555</wheel_separation>
-      <wheel_radius>0.165</wheel_radius>
+      <wheel_separation>0.835</wheel_separation>
+      <wheel_radius>0.145</wheel_radius>
       <!-- Topics / frames -->
       <topic>/cmd_vel</topic>
