Commit message: change box pose

File: ros_ws/src/hs_description/model/Assemblies/Rig6/model.sdf.xacro (robot description, xacro)
@@ -38,5 +38,5 @@
       <pose relative_to="top_plate_link">${rig_pos_relative_2_joint}</pose>
     </link>
-    <xacro:Rig_simpelBox_xacro size="${box_size_x} ${box_size_y} ${box_size_z}" offset="${rig_pos_relative_2_joint}"/>
+    <xacro:Rig_simpelBox_xacro size="${box_size_x} ${box_size_y} ${box_size_z}" offset="${rig_pos_relative_2_joint}" base_frame="rig_link"/>
     <!--use box_size_x,box_size_y,box_size_z in the offset to allign sensor placement-->
     <!-- <origin xyz="${oakd_x_offset} ${oakd_y_offset} ${oakd_z_offset}"/> -->

File: ros_ws/src/hs_description/model/Rigs/Rig_simpelBox_xacro/model.sdf.xacro (robot description, xacro)
@@ -1,7 +1,8 @@
 <?xml version="1.0" ?>
-  <sdf version="1.10" xmlns:xacro="http://www.ros.org/wiki/xacro">
-    <xacro:macro name="Rig_simpelBox_xacro" params='size:="0.6 0.4 0.5" offset:="0 0 0 0 0 0"'>
+<sdf version="1.10" xmlns:xacro="http://www.ros.org/wiki/xacro">
+  <xacro:macro name="Rig_simpelBox_xacro" params='size:="0.6 0.4 0.5" offset:="0 0 0 0 0 0" base_frame'>
     <static>false</static>
     <link name="box_link">
+      <pose relative_to="${base_frame}">0 0 0 0 0 0</pose>
       <gravity>true</gravity>
       <collision name="c">
@@ -10,6 +11,12 @@
       <visual name="v">
         <geometry><box><size>${size}</size></box></geometry>
+        <material>
+          <ambient>0.2 0.2 0.2 1</ambient>
+          <diffuse>0.8 0.1 0.1 1</diffuse>
+          <specular>0.5 0.5 0.5 1</specular>
+          <emissive>0 0 0 1</emissive>
+        </material>
       </visual>
     </link>
-    </xacro:macro>
-  </sdf>
+  </xacro:macro>
+</sdf>
