Commit message: add imu plugin to simulation
- initialize gazebo IMU plugin in worlds
- add IMU to livox lidar
- add livox lidar's IMU to gz bridge
- change IMU pose in oakd to reflect its actual position

File: ros_ws/src/s_description/model/Sensors/mid360_lidar/model.sdf.xacro (robot description, xacro)
@@ -3,8 +3,8 @@
   <xacro:macro name="mid360_lidar" params='name:=mid360_lidar parent_link xyz:="0 0 0" rpy:="0 0 0"'>
     <xacro:property name="base_frame" value="${name}_link"/>
-      <link name="${base_frame}">
-        <pose relative_to="${parent_link}">${xyz} ${rpy}</pose>
-        <gravity>true</gravity>
-        <visual name="Lidar_vizual_1">
+    <link name="${base_frame}">
+      <pose relative_to="${parent_link}">${xyz} ${rpy}</pose>
+      <gravity>true</gravity>
+      <visual name="Lidar_vizual_1">
         <pose relative_to="${base_frame}">0 0 0 ${pi/2} 0 0</pose>
         <geometry>
@@ -26,42 +26,72 @@
         </geometry>
       </collision>
-        <sensor name="mid360_like" type="gpu_lidar">
-                <visualize>true</visualize>
-                <always_on>1</always_on>
-                <update_rate>10</update_rate>
-                <lidar>
-                  <scan>
-                    <horizontal>
-                      <samples>720</samples>  <!-- MID-360 0.5° resolution -->
-                      <resolution>1</resolution>
-                      <min_angle>-3.14156</min_angle>
-                      <max_angle>3.14156</max_angle>
-                    </horizontal>
-                    <vertical>
-                      <samples>40</samples>
-                      <resolution>1</resolution>
-                      <min_angle>-0.122173048555</min_angle> <!-- -7° -->
-                      <max_angle>0.907571211037</max_angle>  <!-- +52° -->
-                    </vertical>
-                  </scan>
-                  <range>
-                    <min>0.10</min> <!-- MID-360 blind zone ~0.1 m -->
-                    <max>40</max>
-                    <resolution>0.01</resolution>
-                  </range>
-                  <noise>
-                    <type>gaussian</type>
-                    <mean>0.0</mean>
-                    <stddev>0.02</stddev>
-                  </noise>
-                </lidar>
-                <topic>/lidar_points</topic>  <!-- Gazebo Transport topic -->
-                <pose relative_to="${base_frame}">0 0 0 0 0 0</pose>
-          </sensor>
-      </link>
-      <joint name="mid360_lidar_mount" type="fixed">
-        <parent>${parent_link}</parent>
-        <child>${base_frame}</child>
-      </joint>
+      <sensor name="mid360_like" type="gpu_lidar">
+        <visualize>true</visualize>
+        <always_on>1</always_on>
+        <update_rate>10</update_rate>
+        <lidar>
+          <scan>
+            <horizontal>
+              <samples>720</samples>  <!-- MID-360 0.5° resolution -->
+              <resolution>1</resolution>
+              <min_angle>-3.14156</min_angle>
+              <max_angle>3.14156</max_angle>
+            </horizontal>
+            <vertical>
+              <samples>40</samples>
+              <resolution>1</resolution>
+              <min_angle>-0.122173048555</min_angle> <!-- -7° -->
+              <max_angle>0.907571211037</max_angle>  <!-- +52° -->
+            </vertical>
+          </scan>
+          <range>
+            <min>0.10</min> <!-- MID-360 blind zone ~0.1 m -->
+            <max>40</max>
+            <resolution>0.01</resolution>
+          </range>
+          <noise>
+            <type>gaussian</type>
+            <mean>0.0</mean>
+            <stddev>0.02</stddev>
+          </noise>
+        </lidar>
+        <topic>/lidar_points</topic>  <!-- Gazebo Transport topic -->
+        <pose relative_to="${base_frame}">0 0 0 0 0 0</pose>
+      </sensor>
+    </link>
+    <joint name="mid360_lidar_mount" type="fixed">
+      <parent>${parent_link}</parent>
+      <child>${base_frame}</child>
+    </joint>
+    <link name="${name}_imu_frame">
+      <xacro:inertial_dummy/>
+      <sensor name="${name}_imu_sensor" type="imu">
+        <always_on>1</always_on>
+        <update_rate>100</update_rate>
+        <imu>
+          <angular_velocity>
+            <noise>
+              <type>gaussian</type>
+              <mean>0.0</mean>
+              <stddev>0.001</stddev>
+            </noise>
+          </angular_velocity>
+          <linear_acceleration>
+            <noise>
+              <type>gaussian</type>
+              <mean>0.0</mean>
+              <stddev>0.02</stddev>
+            </noise>
+          </linear_acceleration>
+        </imu>
+        <topic>/livox/imu</topic>
+        <gz_frame_id>${name}_imu_frame</gz_frame_id>
+      </sensor>
+    </link>
+    <joint name="${name}_imu_joint" type="fixed">
+      <parent>${base_frame}</parent>
+      <child>${name}_imu_frame</child>
+      <pose relative_to="${base_frame}">0 0 0 0 0 0</pose>
+    </joint>
   </xacro:macro>
 </sdf>

File: ros_ws/src/s_description/model/Sensors/oakd/model.sdf.xacro (robot description, xacro)
@@ -190,4 +190,5 @@
             </orientation>
           </imu>
+          <pose relative_to="${base_frame}">0 0 0 ${M_PI/2} 0 ${M_PI/2}</pose>
           <topic>/oakd/imu</topic>
           <gz_frame_id>${name}_imu_frame</gz_frame_id>
