Commit message: fixed vlads pull request comments

File: ros_ws/src/s_description/model/Assemblies/Rig5/model.sdf.xacro (robot description, xacro)
@@ -12,5 +12,5 @@
     <xacro:property name="mid360_lidar_x_offset" value="${0*cm2m}"/>
     <xacro:property name="mid360_lidar_y_offset" value="${0*cm2m}"/>
-    <xacro:property name="mid360_lidar_z_offset" value="${0*cm2m}"/>
+    <xacro:property name="mid360_lidar_z_offset" value="${3*cm2m}"/>
     <xacro:property name="rig_pos_relative_2_UGV" value="0 0 0.45 0 0 0"/>
     <xacro:property name="gnss_x_offset" value="${0*cm2m}"/>

File: ros_ws/src/s_description/model/Sensors/mid360_lidar/model.sdf.xacro (robot description, xacro)
@@ -7,60 +7,20 @@
         <gravity>true</gravity>
         <visual name="Lidar_vizual_1">
-        <pose relative_to="${base_frame}">0 0 0 0 0 0</pose>
+        <pose relative_to="${base_frame}">0 0 0 ${pi/2} 0 0</pose>
         <geometry>
           <mesh>
             <scale>1 1 1</scale>
             <!-- <uri>meshes/VLP16_base_1.dae</uri>-->
-            <uri>model://mid360_lidar/meshes/VLP16_base_1.dae</uri>
+            <uri>model://mid360_lidar/meshes/MID_360.dae</uri>
           </mesh>
         </geometry>
       </visual>
       <collision name="Lidar_collision_1">
-        <pose relative_to="${base_frame}">0 0 0 0 0 0</pose>
+        <pose relative_to="${base_frame}">0 0 0 ${pi/2} 0 0</pose>
         <geometry>
           <mesh>
             <scale>1 1 1</scale>
             <!--<uri>meshes/VLP16_base_1.dae</uri>-->
-            <uri>model://mid360_lidar/meshes/VLP16_base_1.dae</uri>
-          </mesh>
-        </geometry>
-      </collision>
-      <visual name="Lidar_vizual_2">
-        <pose relative_to="${base_frame}">0 0 0 0 0 0</pose>
-        <geometry>
-          <mesh>
-            <scale>1 1 1</scale>
-            <!--<uri>meshes/VLP16_base_2.dae</uri>-->
-            <uri>model://mid360_lidar/meshes/VLP16_base_2.dae</uri>
-          </mesh>
-        </geometry>
-      </visual>
-      <collision name="Lidar_collision_2">
-        <pose relative_to="${base_frame}">0 0 0 0 0 0</pose>
-        <geometry>
-          <mesh>
-            <scale>1 1 1</scale>
-            <!--<uri>meshes/VLP16_base_2.dae</uri>-->
-            <uri>model://mid360_lidar/meshes/VLP16_base_2.dae</uri>
-          </mesh>
-        </geometry>
-      </collision>
-      <visual name="Lidar_vizual_3">
-        <pose relative_to="${base_frame}">0 0 0 0 0 0</pose>
-        <geometry>
-          <mesh>
-            <scale>1 1 1</scale>
-            <!--<uri>meshes/VLP16_scan.dae</uri>-->
-            <uri>model://mid360_lidar/meshes/VLP16_scan.dae</uri>
-          </mesh>
-        </geometry>
-      </visual>
-      <collision name="Lidar_collision_3">
-        <pose relative_to="${base_frame}">0 0 0 0 0 0</pose>
-        <geometry>
-          <mesh>
-            <scale>1 1 1</scale>
-            <!--<uri>meshes/VLP16_scan.dae</uri>-->
-            <uri>model://mid360_lidar/meshes/VLP16_scan.dae</uri>
+            <uri>model://mid360_lidar/meshes/MID_360.dae</uri>
           </mesh>
         </geometry>

Commit message: updated the model Assembly  framework to match the one Vlad had implemented in hs_description to give more control from the Assembly file

File: ros_ws/src/s_description/model/Assemblies/Rig5/model.sdf.xacro (robot description, xacro)
@@ -17,4 +17,7 @@
     <xacro:property name="gnss_y_offset" value="${0*cm2m}"/>
     <xacro:property name="gnss_z_offset" value="${15*cm2m}"/>
+    <xacro:property name="box_size_x" value="0.6"/>
+    <xacro:property name="box_size_y" value="0.4"/>
+    <xacro:property name="box_size_z" value="0.5"/>
     <link name="rig_link">
       <inertial>
@@ -27,5 +30,5 @@
       <pose relative_to="UGV_link">${rig_pos_relative_2_UGV}</pose>
     </link>
-    <xacro:Rig_simpelBox_xacro UGV_link="UGV_link" offset="${rig_pos_relative_2_UGV}"/>
+    <xacro:Rig_simpelBox_xacro base_frame="rig_link" size="${box_size_x} ${box_size_y} ${box_size_z}" offset="${rig_pos_relative_2_UGV}"/>
     <!--use box_size_x,box_size_y,box_size_z in the offset to allign sensor placement-->
     <!-- <origin xyz="${oakd_x_offset} ${oakd_y_offset} ${oakd_z_offset}"/> -->
@@ -84,5 +87,4 @@
       <child>rig_link</child>
     </joint>
-    <pose>0 0 0 0 0 0</pose>
   </model>
 </sdf>

File: ros_ws/src/s_description/model/Assemblies/Rig7/model.sdf.xacro (robot description, xacro)
@@ -17,4 +17,7 @@
     <xacro:property name="gnss_y_offset" value="${0*cm2m}"/>
     <xacro:property name="gnss_z_offset" value="${15*cm2m}"/>
+    <xacro:property name="box_size_x" value="0.6"/>
+    <xacro:property name="box_size_y" value="0.4"/>
+    <xacro:property name="box_size_z" value="0.5"/>
     <link name="rig_link">
       <inertial>
@@ -27,5 +30,5 @@
       <pose relative_to="UGV_link">${rig_pos_relative_2_UGV}</pose>
     </link>
-    <xacro:Rig_simpelBox_xacro UGV_link="UGV_link" offset="${rig_pos_relative_2_UGV}"/>
+    <xacro:Rig_simpelBox_xacro base_frame="rig_link" size="${box_size_x} ${box_size_y} ${box_size_z}" offset="${rig_pos_relative_2_UGV}"/>
     <!--use box_size_x,box_size_y,box_size_z in the offset to allign sensor placement-->
     <!-- <origin xyz="${oakd_x_offset} ${oakd_y_offset} ${oakd_z_offset}"/> -->
@@ -84,5 +87,4 @@
       <child>rig_link</child>
     </joint>
-    <pose>0 0 0 0 0 0</pose>
   </model>
 </sdf>

File: ros_ws/src/s_description/model/Rigs/Rig_simpelBox_xacro/model.sdf.xacro (robot description, xacro)
@@ -1,20 +1,22 @@
 <?xml version="1.0" ?>
-  <sdf version="1.10" xmlns:xacro="http://www.ros.org/wiki/xacro">
-      <!-- Parameters -->
-  <xacro:property name="box_size_x" value="0.6"/>
-  <xacro:property name="box_size_y" value="0.4"/>
-  <xacro:property name="box_size_z" value="0.5"/>
-    <xacro:macro name="Rig_simpelBox_xacro" params='offset:="0 0 0 0 0 0" UGV_link'>
+<sdf version="1.10" xmlns:xacro="http://www.ros.org/wiki/xacro">
+  <xacro:macro name="Rig_simpelBox_xacro" params='size:="0.6 0.4 0.5" offset:="0 0 0 0 0 0" base_frame'>
     <static>false</static>
     <link name="box_link">
-      <pose>${offset}</pose>
+      <pose relative_to="${base_frame}">0 0 0 0 0 0</pose>
       <gravity>true</gravity>
       <collision name="c">
-        <geometry><box><size>${box_size_x} ${box_size_y} ${box_size_z}</size></box></geometry>
+        <geometry><box><size>${size}</size></box></geometry>
       </collision>
       <visual name="v">
-        <geometry><box><size>${box_size_x} ${box_size_y} ${box_size_z}</size></box></geometry>
+        <geometry><box><size>${size}</size></box></geometry>
+        <material>
+          <ambient>0.2 0.2 0.2 1</ambient>
+          <diffuse>0.8 0.1 0.1 1</diffuse>
+          <specular>0.5 0.5 0.5 1</specular>
+          <emissive>0 0 0 1</emissive>
+        </material>
       </visual>
     </link>
-    </xacro:macro>
-  </sdf>
+  </xacro:macro>
+</sdf>

File: ros_ws/src/s_description/model/Sensors/mid360_lidar/model.sdf.xacro (robot description, xacro)
@@ -2,5 +2,5 @@
 <sdf version="1.10" xmlns:xacro="http://ros.org/wiki/xacro">
   <xacro:macro name="mid360_lidar" params='name:=mid360_lidar parent_link xyz:="0 0 0" rpy:="0 0 0"'>
-    <xacro:property name="base_frame" value="${name}_link"/>
+    <xacro:property name="base_frame" value="livox_frame"/>
     <link name="${base_frame}">
       <pose relative_to="${parent_link}">${xyz} ${rpy}</pose>
@@ -92,5 +92,4 @@
       <parent>${base_frame}</parent>
       <child>${name}_imu_frame</child>
-      <pose relative_to="${base_frame}">0 0 0 0 0 0</pose>
     </joint>
   </xacro:macro>
