Commit message: test description on husky

File: ros_ws/src/hs_description/model/Assemblies/Rig5/model.sdf.xacro (robot description, xacro)
@@ -6,5 +6,5 @@
   <xacro:include filename="$(find hs_description)/model/UGV/Husky_stripped_xacro/model.sdf.xacro"/>
   <xacro:include filename="$(find hs_description)/model/Sensors/navsat_gnss/model.sdf.xacro"/>
-  <model name="Rig5" canonical_link='UGV_link'>
+  <model name="Rig5" canonical_link='base_link'>
     <xacro:property name="oakd_x_offset" value="${4*cm2m}"/>
     <xacro:property name="oakd_y_offset" value="${0*cm2m}"/>
@@ -25,7 +25,7 @@
       </inertia>
       </inertial>
-      <pose relative_to="UGV_link">${rig_pos_relative_2_UGV}</pose>
+      <pose relative_to="base_link">${rig_pos_relative_2_UGV}</pose>
     </link>
-    <xacro:Rig_simpelBox_xacro UGV_link="UGV_link" offset="${rig_pos_relative_2_UGV}"/>
+    <xacro:Rig_simpelBox_xacro UGV_link="base_link" offset="${rig_pos_relative_2_UGV}"/>
     <!--use box_size_x,box_size_y,box_size_z in the offset to allign sensor placement-->
     <!-- <origin xyz="${oakd_x_offset} ${oakd_y_offset} ${oakd_z_offset}"/> -->
@@ -50,6 +50,6 @@
     <xacro:navsat_gnss parent_link="rig_top_link" xyz="${gnss_x_offset} ${gnss_y_offset} ${gnss_z_offset}" rpy="0 0 0"/>
     <xacro:oakd parent_link="rig_front_link" xyz="${oakd_x_offset} ${oakd_y_offset} ${oakd_z_offset}" rpy="0 0 0"/>
-    <xacro:mid360_lidar parent_link="rig_top_link" xyz="${mid360_lidar_x_offset} ${mid360_lidar_y_offset} ${mid360_lidar_z_offset}" rpy="0 0 0"/>
-    <xacro:Husky_stripped_xacro base_link="UGV_link"/>
+    <xacro:mid360_lidar parent_link="rig_top_link" xyz="${mid360_lidar_x_offset} ${mid360_lidar_y_offset} ${mid360_lidar_z_offset}" rpy="0 0 ${pi}"/>
+    <xacro:Husky_stripped_xacro base_link="base_link"/>
     <joint name="base_joint" type="fixed">
       <parent>rig_link</parent>
@@ -81,5 +81,5 @@
     </joint>
     <joint name="UGV_rig_mount" type="fixed">
-      <parent>UGV_link</parent>
+      <parent>base_link</parent>
       <child>rig_link</child>
     </joint>

File: ros_ws/src/hs_description/model/Sensors/mid360_lidar/model.sdf.xacro (robot description, xacro)
@@ -2,5 +2,5 @@
 <sdf version="1.10" xmlns:xacro="http://ros.org/wiki/xacro">
   <xacro:macro name="mid360_lidar" params='name:=mid360_lidar parent_link xyz:="0 0 0" rpy:="0 0 0"'>
-    <xacro:property name="base_frame" value="${name}_link"/>
+    <xacro:property name="base_frame" value="livox_frame"/>
       <link name="${base_frame}">
         <pose relative_to="${parent_link}">${xyz} ${rpy}</pose>

Commit message: backport to Rig5

File: ros_ws/src/hs_description/model/Assemblies/Rig5/model.sdf.xacro (robot description, xacro)
@@ -17,4 +17,7 @@
     <xacro:property name="gnss_y_offset" value="${0*cm2m}"/>
     <xacro:property name="gnss_z_offset" value="${15*cm2m}"/>
+    <xacro:property name="box_size_x" value="0.6"/>
+    <xacro:property name="box_size_y" value="0.4"/>
+    <xacro:property name="box_size_z" value="0.5"/>
     <link name="rig_link">
       <inertial>
@@ -27,5 +30,5 @@
       <pose relative_to="UGV_link">${rig_pos_relative_2_UGV}</pose>
     </link>
-    <xacro:Rig_simpelBox_xacro UGV_link="UGV_link" offset="${rig_pos_relative_2_UGV}"/>
+    <xacro:Rig_simpelBox_xacro base_frame="rig_link" size="${box_size_x} ${box_size_y} ${box_size_z}" offset="${rig_pos_relative_2_UGV}"/>
     <!--use box_size_x,box_size_y,box_size_z in the offset to allign sensor placement-->
     <!-- <origin xyz="${oakd_x_offset} ${oakd_y_offset} ${oakd_z_offset}"/> -->
@@ -84,5 +87,4 @@
       <child>rig_link</child>
     </joint>
-    <pose>0 0 0 0 0 0</pose>
   </model>
 </sdf>

Commit message: test setup with chair
- use fast_lio instead of wheel odometry
- change rotation of the lidar in the driver config instead of urdf
- change the rotation vector type in oakd config
- exclude GPS from odometry (for now)

File: ros_ws/src/hs_description/model/Assemblies/Rig5/model.sdf.xacro (robot description, xacro)
@@ -53,5 +53,5 @@
     <xacro:navsat_gnss parent_link="rig_top_link" xyz="${gnss_x_offset} ${gnss_y_offset} ${gnss_z_offset}" rpy="0 0 0"/>
     <xacro:oakd parent_link="rig_front_link" xyz="${oakd_x_offset} ${oakd_y_offset} ${oakd_z_offset}" rpy="0 0 0"/>
-    <xacro:mid360_lidar parent_link="rig_top_link" xyz="${mid360_lidar_x_offset} ${mid360_lidar_y_offset} ${mid360_lidar_z_offset}" rpy="0 0 ${pi}"/>
+    <xacro:mid360_lidar parent_link="rig_top_link" xyz="${mid360_lidar_x_offset} ${mid360_lidar_y_offset} ${mid360_lidar_z_offset}" rpy="0 0 0"/>
     <xacro:Husky_stripped_xacro base_link="base_link"/>
     <joint name="base_joint" type="fixed">

File: ros_ws/src/hs_description/model/Sensors/oakd/model.sdf.xacro (robot description, xacro)
@@ -2,5 +2,5 @@
 <sdf version="1.11" xmlns:xacro="http://ros.org/wiki/xacro">
   <xacro:include filename="$(find hs_description)/model/Sensors/oakd/common.sdf.xacro" />
-    <xacro:macro name="oakd" params='name:=oakd_pro parent_link xyz:="0 0 0" rpy:="0 0 0"'>
+    <xacro:macro name="oakd" params='name:=oakd parent_link xyz:="0 0 0" rpy:="0 0 0"'>
       <xacro:property name="mass"       value="0.061"/>
       <xacro:property name="baseline"   value="0.075" />

Commit message: description changes

File: ros_ws/src/hs_description/model/Assemblies/Rig5/model.sdf.xacro (robot description, xacro)
@@ -7,5 +7,5 @@
   <xacro:include filename="$(find hs_description)/model/Sensors/navsat_gnss/model.sdf.xacro"/>
   <model name="Rig5" canonical_link='base_link'>
-    <xacro:property name="oakd_x_offset" value="${4*cm2m}"/>
+    <xacro:property name="oakd_x_offset" value="${30*cm2m}"/>
     <xacro:property name="oakd_y_offset" value="${0*cm2m}"/>
     <xacro:property name="oakd_z_offset" value="${0*cm2m}"/>
@@ -52,6 +52,6 @@
     </link>
     <xacro:navsat_gnss parent_link="rig_top_link" xyz="${gnss_x_offset} ${gnss_y_offset} ${gnss_z_offset}" rpy="0 0 0"/>
-    <xacro:oakd parent_link="rig_front_link" xyz="${oakd_x_offset} ${oakd_y_offset} ${oakd_z_offset}" rpy="0 0 0"/>
-    <xacro:mid360_lidar parent_link="rig_top_link" xyz="${mid360_lidar_x_offset} ${mid360_lidar_y_offset} ${mid360_lidar_z_offset}" rpy="0 0 0"/>
+    <xacro:oakd parent_link="rig_link" xyz="${oakd_x_offset} ${oakd_y_offset} ${oakd_z_offset}" rpy="0 ${pi/6} 0"/>
+    <xacro:mid360_lidar parent_link="rig_link" xyz="${mid360_lidar_x_offset} ${mid360_lidar_y_offset} ${mid360_lidar_z_offset}" rpy="0 0 0"/>
     <xacro:Husky_stripped_xacro base_link="base_link"/>
     <joint name="base_joint" type="fixed">
