Commit message: Fixed comments by Vlad

File: ros_ws/src/s_description/model/Assemblies/Rig6/model.sdf.xacro (robot description, xacro)
@@ -40,5 +40,4 @@
     <xacro:Rig_simpelBox_xacro size="${box_size_x} ${box_size_y} ${box_size_z}" offset="${rig_pos_relative_2_joint}" base_frame="rig_link"/>
     <!--use box_size_x,box_size_y,box_size_z in the offset to allign sensor placement-->
-    <!-- <origin xyz="${oakd_x_offset} ${oakd_y_offset} ${oakd_z_offset}"/> -->
     <link name="rig_bottom_link">
       <pose relative_to="rig_link">0 0 ${-0.5*box_size_z} 0 0 0</pose>
@@ -94,5 +93,4 @@
       <parent>top_plate_link</parent>
       <child>rig_link</child>
-      <!-- <pose relative_to="top_plate_link">${rig_pos_relative_2_joint}</pose> -->
     </joint>
   </model>

File: ros_ws/src/s_description/model/Rigs/Rig_simpelBox_xacro/model.sdf.xacro (robot description, xacro)
@@ -4,5 +4,5 @@
     <static>false</static>
     <link name="box_link">
-      <pose relative_to="${base_frame}">0 0 0 0 0 0</pose>
+      <pose relative_to="${base_frame}">${offset}</pose>
       <gravity>true</gravity>
       <collision name="c">

File: ros_ws/src/s_description/model/UGV/Light_seeker/model.sdf.xacro (robot description, xacro)
@@ -27,5 +27,4 @@
         </geometry>
       </visual>
-    </link>
       <velocity_decay/>
       <self_collide>0</self_collide>
@@ -34,4 +33,5 @@
       <gravity>1</gravity>
       <velocity_decay/>
+    </link>
     <link name="base_footprint">
       <pose frame="">0 0 -0.33 0 0 0</pose>
