Commit message: Changed rig7 configuration to estimate real model (untested)

File: ros_ws/src/s_description/model/Assemblies/Rig7/model.sdf.xacro (robot description, xacro)
@@ -13,11 +13,11 @@
     <xacro:property name="mid360_lidar_y_offset" value="${0*cm2m}"/>
     <xacro:property name="mid360_lidar_z_offset" value="${3*cm2m}"/>
-    <xacro:property name="rig_pos_relative_2_UGV" value="0 0 ${0.19/2+0.17/2} 0 0 0"/>
     <xacro:property name="gnss_x_offset" value="${0*cm2m}"/>
     <xacro:property name="gnss_y_offset" value="${0*cm2m}"/>
     <xacro:property name="gnss_z_offset" value="${15*cm2m}"/>
-    <xacro:property name="box_size_x" value="0.6"/>
-    <xacro:property name="box_size_y" value="0.4"/>
-    <xacro:property name="box_size_z" value="0.5"/>
+    <xacro:property name="box_size_x" value="0.1"/>
+    <xacro:property name="box_size_y" value="0.1"/>
+    <xacro:property name="box_size_z" value="0.25"/>
+    <xacro:property name="rig_pos_relative_2_UGV" value="0 0 ${0.19/2+0.17/2} 0 0 0"/>
     <link name="rig_link">
       <inertial>

Commit message: fixed the sensor rig to match the current configuration

File: ros_ws/src/s_description/model/Assemblies/Rig7/model.sdf.xacro (robot description, xacro)
@@ -7,7 +7,13 @@
   <xacro:include filename="$(find s_description)/model/Sensors/navsat_gnss/model.sdf.xacro"/>
   <model name="Rig7" canonical_link='UGV_link'>
-    <xacro:property name="oakd_x_offset" value="${4*cm2m}"/>
-    <xacro:property name="oakd_y_offset" value="${0*cm2m}"/>
-    <xacro:property name="oakd_z_offset" value="${0*cm2m}"/>
+    <xacro:property name="box_size_x" value="${6.4*cm2m}"/>
+    <xacro:property name="box_size_y" value="${6.4*cm2m}"/>
+    <xacro:property name="box_size_z" value="${25*cm2m}"/>
+    <xacro:property name="oakd_1_x_offset" value="${(1.3+2.8/2)*cm2m}"/>
+    <xacro:property name="oakd_1_y_offset" value="${0*cm2m}"/>
+    <xacro:property name="oakd_1_z_offset" value="${(25/2-1.3)*cm2m}"/>
+    <xacro:property name="oakd_2_x_offset" value="${(1.3+2.8/2)*cm2m}"/>
+    <xacro:property name="oakd_2_y_offset" value="${0*cm2m}"/>
+    <xacro:property name="oakd_2_z_offset" value="${(25/2-1.3)*cm2m}"/>
     <xacro:property name="mid360_lidar_x_offset" value="${0*cm2m}"/>
     <xacro:property name="mid360_lidar_y_offset" value="${0*cm2m}"/>
@@ -15,8 +21,5 @@
     <xacro:property name="gnss_x_offset" value="${0*cm2m}"/>
     <xacro:property name="gnss_y_offset" value="${0*cm2m}"/>
-    <xacro:property name="gnss_z_offset" value="${15*cm2m}"/>
-    <xacro:property name="box_size_x" value="0.1"/>
-    <xacro:property name="box_size_y" value="0.1"/>
-    <xacro:property name="box_size_z" value="0.25"/>
+    <xacro:property name="gnss_z_offset" value="${0*cm2m}"/>
     <xacro:property name="rig_pos_relative_2_UGV" value="0 0 ${0.19/2+0.17/2} 0 0 0"/>
     <link name="rig_link">
@@ -52,5 +55,6 @@
     </link>
     <xacro:navsat_gnss parent_link="rig_top_link" xyz="${gnss_x_offset} ${gnss_y_offset} ${gnss_z_offset}" rpy="0 0 0"/>
-    <xacro:oakd parent_link="rig_front_link" xyz="${oakd_x_offset} ${oakd_y_offset} ${oakd_z_offset}" rpy="0 0 0"/>
+    <xacro:oakd parent_link="rig_front_link" name="oakd_pro_1" xyz="${oakd_1_x_offset} ${oakd_1_y_offset} ${oakd_1_z_offset}" rpy="0 ${pi/180*15} 0"/>
+    <xacro:oakd parent_link="rig_back_link" name="oakd_pro_2" xyz="${-oakd_2_x_offset} ${oakd_2_y_offset} ${oakd_2_z_offset}" rpy="0 ${pi/180*15} ${pi}"/>
     <xacro:mid360_lidar parent_link="rig_top_link" xyz="${mid360_lidar_x_offset} ${mid360_lidar_y_offset} ${mid360_lidar_z_offset}" rpy="0 0 0"/>
     <xacro:Light_seeker base_link="UGV_link"/>

File: ros_ws/src/s_description/model/Sensors/oakd/model.sdf.xacro (robot description, xacro)
@@ -71,5 +71,5 @@
             </clip>
           </depth_camera>
-          <topic>/oakd/rgbd</topic>
+          <topic>${name}/oakd/rgbd</topic>
           <gz_frame_id>${name}_rgb_camera_frame</gz_frame_id>
         </sensor>
@@ -83,8 +83,11 @@
       </link>
       <joint name="${name}_rgb_camera_optical_joint" type="fixed">
+        <pose relative_to="${name}_rgb_camera_frame">0 0 0 -${M_PI/2} 0.0 -${M_PI/2}</pose>
         <parent>${name}_rgb_camera_frame</parent>
         <child>${name}_rgb_camera_optical_frame</child>
       </joint>
-      <link name="${name}_rgb_camera_sensor_mount" />
+      <link name="${name}_rgb_camera_sensor_mount">
+        <pose relative_to="${base_frame}">0 0 0 0 0 0</pose>
+      </link>
       <joint name="${name}_rgb_camera_sensor_mount_joint" type="fixed">
         <parent>${name}_rgb_camera_optical_frame</parent>
@@ -94,4 +97,5 @@
       <link name="${name}_left_camera_frame">
         <xacro:inertial_dummy/>
+        <pose relative_to="${base_frame}">0 ${baseline/2} 0 0 0 0</pose>
         <sensor name="${name}_left_camera_sensor" type="camera">
           <always_on>1</always_on>
@@ -109,5 +113,5 @@
             </clip>
           </camera>
-          <topic>/oakd/left</topic>
+          <topic>${name}/oakd/left</topic>
           <gz_frame_id>${name}_left_camera_frame</gz_frame_id>
         </sensor>
@@ -116,11 +120,10 @@
         <parent>${base_frame}</parent>
         <child>${name}_left_camera_frame</child>
-        <pose relative_to="${base_frame}">0 ${baseline/2} 0 0 0 0</pose>
       </joint>
       <link name="${name}_left_camera_optical_frame">
         <xacro:inertial_dummy/>
+        <pose relative_to="${name}_left_camera_frame">0 0 0 -${M_PI/2} 0.0 -${M_PI/2}</pose>
       </link>
       <joint name="${name}_left_camera_optical_joint" type="fixed">
-        <pose relative_to="${base_frame}">0 0 0 -${M_PI/2} 0.0 -${M_PI/2}</pose>
         <parent>${name}_left_camera_frame</parent>
         <child>${name}_left_camera_optical_frame</child>
@@ -129,4 +132,5 @@
       <link name="${name}_right_camera_frame">
         <xacro:inertial_dummy/>
+        <pose relative_to="${base_frame}">0 -${baseline/2} 0 0 0 0</pose>
         <sensor name="${name}_right_camera_sensor" type="camera">
           <always_on>1</always_on>
@@ -144,5 +148,5 @@
             </clip>
           </camera>
-          <topic>/oakd/right</topic>
+          <topic>${name}/oakd/right</topic>
           <gz_frame_id>${name}_right_camera_frame</gz_frame_id>
         </sensor>
@@ -151,11 +155,10 @@
         <parent>${base_frame}</parent>
         <child>${name}_right_camera_frame</child>
-        <pose relative_to="${base_frame}">0 -${baseline/2} 0 0 0 0</pose>
       </joint>
       <link name="${name}_right_camera_optical_frame">
         <xacro:inertial_dummy/>
+        <pose relative_to="${name}_right_camera_frame">0 0 0 -${M_PI/2} 0.0 -${M_PI/2}</pose>
       </link>
       <joint name="${name}_right_camera_optical_joint" type="fixed">
-        <pose relative_to="${base_frame}">0 0 0 -${M_PI/2} 0.0 -${M_PI/2}</pose>
         <parent>${name}_right_camera_frame</parent>
         <child>${name}_right_camera_optical_frame</child>
@@ -191,5 +194,5 @@
           </imu>
           <pose relative_to="${base_frame}">0 0 0 ${M_PI/2} 0 ${M_PI/2}</pose>
-          <topic>/oakd/imu</topic>
+          <topic>${name}/oakd/imu</topic>
           <gz_frame_id>${name}_imu_frame</gz_frame_id>
         </sensor>
@@ -198,7 +201,6 @@
         <parent>${base_frame}</parent>
         <child>${name}_imu_frame</child>
-        <pose relative_to="${base_frame}">0 0 0 -${M_PI/2} 0 -${M_PI/2}</pose>
-      </joint>
-      <joint name="oakd_mount" type="fixed">
+      </joint>
+      <joint name="${name}_mount" type="fixed">
         <parent>${parent_link}</parent>
         <child>${base_frame}</child>

Commit message: added README in s_description and did minor changes to ugv

File: ros_ws/src/s_description/model/Assemblies/Rig7/model.sdf.xacro (robot description, xacro)
@@ -57,5 +57,5 @@
     <xacro:oakd parent_link="rig_front_link" name="oakd_pro_1" xyz="${oakd_1_x_offset} ${oakd_1_y_offset} ${oakd_1_z_offset}" rpy="0 ${pi/180*15} 0"/>
     <xacro:oakd parent_link="rig_back_link" name="oakd_pro_2" xyz="${-oakd_2_x_offset} ${oakd_2_y_offset} ${oakd_2_z_offset}" rpy="0 ${pi/180*15} ${pi}"/>
-    <xacro:mid360_lidar parent_link="rig_top_link" xyz="${mid360_lidar_x_offset} ${mid360_lidar_y_offset} ${mid360_lidar_z_offset}" rpy="0 0 0"/>
+    <xacro:mid360_lidar parent_link="rig_top_link" xyz="${mid360_lidar_x_offset} ${mid360_lidar_y_offset} ${mid360_lidar_z_offset}" rpy="0 0 ${pi/2}"/>
     <xacro:Light_seeker base_link="UGV_link"/>
     <joint name="base_joint" type="fixed">

File: ros_ws/src/s_description/model/UGV/Light_seeker/model.sdf.xacro (robot description, xacro)
@@ -1,8 +1,8 @@
 <?xml version='1.0' encoding='utf-8'?>
 <sdf version="1.6" xmlns:xacro="http://www.ros.org/wiki/xacro">
-  <xacro:macro name="Light_seeker" params='base_link:="base_link"'>
+  <xacro:macro name="Light_seeker" params='base_link'>
     <xacro:property name="groundz_z_offset" value="${0.1}"/>
     <link name="${base_link}">
-      <pose frame="">0 0 0 0 0 0</pose>
+      <pose>0 0 0 0 0 0</pose>
       <inertial>
         <pose frame="">0 0 0.062329 0 -0 0</pose>

Commit message: Simulation demo, works but small config values needs to be adjusted

File: ros_ws/src/s_description/model/Assemblies/Rig7/model.sdf.xacro (robot description, xacro)
@@ -6,5 +6,5 @@
   <xacro:include filename="$(find s_description)/model/UGV/Light_seeker/model.sdf.xacro"/>
   <xacro:include filename="$(find s_description)/model/Sensors/navsat_gnss/model.sdf.xacro"/>
-  <model name="Rig7" canonical_link='UGV_link'>
+  <model name="Rig7" canonical_link='base_link'>
     <xacro:property name="box_size_x" value="${6.4*cm2m}"/>
     <xacro:property name="box_size_y" value="${6.4*cm2m}"/>
@@ -18,9 +18,10 @@
     <xacro:property name="mid360_lidar_x_offset" value="${0*cm2m}"/>
     <xacro:property name="mid360_lidar_y_offset" value="${0*cm2m}"/>
-    <xacro:property name="mid360_lidar_z_offset" value="${3*cm2m}"/>
+    <xacro:property name="mid360_lidar_z_offset" value="${0*cm2m}"/>
     <xacro:property name="gnss_x_offset" value="${0*cm2m}"/>
     <xacro:property name="gnss_y_offset" value="${0*cm2m}"/>
     <xacro:property name="gnss_z_offset" value="${0*cm2m}"/>
-    <xacro:property name="rig_pos_relative_2_UGV" value="0 0 ${0.19/2+0.17/2} 0 0 0"/>
+    <!---<xacro:property name="rig_pos_relative_2_UGV" value="0 0 ${0.19/2+0.17/2} 0 0 0"/>  -->
+    <xacro:property name="rig_pos_relative_2_UGV" value="0 0 ${0.19/2+box_size_z/2} 0 0 0"/>
     <link name="rig_link">
       <inertial>
@@ -31,7 +32,7 @@
       </inertia>
       </inertial>
-      <pose relative_to="UGV_link">${rig_pos_relative_2_UGV}</pose>
+      <pose relative_to="base_link">${rig_pos_relative_2_UGV}</pose>
     </link>
-    <xacro:Rig_simpelBox_xacro base_frame="rig_link" size="${box_size_x} ${box_size_y} ${box_size_z}" offset="${rig_pos_relative_2_UGV}"/>
+    <xacro:Rig_simpelBox_xacro base_frame="rig_link" size="${box_size_x} ${box_size_y} ${box_size_z}"/>
     <!--use box_size_x,box_size_y,box_size_z in the offset to allign sensor placement-->
     <!-- <origin xyz="${oakd_x_offset} ${oakd_y_offset} ${oakd_z_offset}"/> -->
@@ -58,5 +59,5 @@
     <xacro:oakd parent_link="rig_back_link" name="oakd_pro_2" xyz="${-oakd_2_x_offset} ${oakd_2_y_offset} ${oakd_2_z_offset}" rpy="0 ${pi/180*15} ${pi}"/>
     <xacro:mid360_lidar parent_link="rig_top_link" xyz="${mid360_lidar_x_offset} ${mid360_lidar_y_offset} ${mid360_lidar_z_offset}" rpy="0 0 ${pi/2}"/>
-    <xacro:Light_seeker base_link="UGV_link"/>
+    <xacro:Light_seeker base_link="base_link"/>
     <joint name="base_joint" type="fixed">
       <parent>rig_link</parent>
@@ -88,5 +89,5 @@
     </joint>
     <joint name="UGV_rig_mount" type="fixed">
-      <parent>UGV_link</parent>
+      <parent>base_link</parent>
       <child>rig_link</child>
     </joint>

File: ros_ws/src/s_description/model/Rigs/Rig_simpelBox_xacro/model.sdf.xacro (robot description, xacro)
@@ -1,8 +1,8 @@
 <?xml version="1.0" ?>
 <sdf version="1.10" xmlns:xacro="http://www.ros.org/wiki/xacro">
-  <xacro:macro name="Rig_simpelBox_xacro" params='size:="0.6 0.4 0.5" offset:="0 0 0 0 0 0" base_frame'>
+  <xacro:macro name="Rig_simpelBox_xacro" params='size:="0.6 0.4 0.5" base_frame'>
     <static>false</static>
     <link name="box_link">
-      <pose relative_to="${base_frame}">${offset}</pose>
+      <pose relative_to="${base_frame}"></pose>
       <gravity>true</gravity>
       <collision name="c">
