Commit message: Minimal model of light_seeker added

File: ros_ws/src/s_description/model/Rigs/Rig_simpelBox_xacro/model.sdf.xacro (robot description, xacro)
@@ -2,7 +2,7 @@
   <sdf version="1.10" xmlns:xacro="http://www.ros.org/wiki/xacro">
       <!-- Parameters -->
-  <xacro:property name="box_size_x" value="0.6"/>
-  <xacro:property name="box_size_y" value="0.4"/>
-  <xacro:property name="box_size_z" value="0.5"/>
+  <xacro:property name="box_size_x" value="0.42"/>
+  <xacro:property name="box_size_y" value="0.38"/>
+  <xacro:property name="box_size_z" value="0.17"/>
     <xacro:macro name="Rig_simpelBox_xacro" params='offset:="0 0 0 0 0 0" UGV_link'>
     <static>false</static>

Commit message: Adding a filter for oakd to ignore points to close, in progress.

File: ros_ws/src/s_description/model/Rigs/Rig_simpelBox_xacro/model.sdf.xacro (robot description, xacro)
@@ -6,7 +6,7 @@
       <pose relative_to="${base_frame}"></pose>
       <gravity>true</gravity>
-      <collision name="c">
+      <!--  <collision name="c">
         <geometry><box><size>${size}</size></box></geometry>
-      </collision>
+      </collision>-->
       <visual name="v">
         <geometry><box><size>${size}</size></box></geometry>

File: ros_ws/src/s_description/model/Sensors/mid360_lidar/model.sdf.xacro (robot description, xacro)
@@ -16,4 +16,5 @@
         </geometry>
       </visual>
+      <!--
       <collision name="Lidar_collision_1">
         <pose relative_to="${base_frame}">0 0 0 ${pi/2} 0 0</pose>
@@ -21,9 +22,9 @@
           <mesh>
             <scale>1 1 1</scale>
-            <!--<uri>meshes/VLP16_base_1.dae</uri>-->
             <uri>model://mid360_lidar/meshes/MID_360.dae</uri>
           </mesh>
         </geometry>
       </collision>
+      -->
       <sensor name="mid360_like" type="gpu_lidar">
         <visualize>true</visualize>

File: ros_ws/src/s_description/model/UGV/Light_seeker/model.sdf.xacro (robot description, xacro)
@@ -27,4 +27,14 @@
         </geometry>
       </visual>
+      <collission name="base_link_visual">
+        <pose frame="">-1.57768 -0.78292 ${-1.12211 - 0.19/2} ${pi/2} 0 ${pi/2}</pose>
+        <!-- Z -X -Y-->
+        <geometry>
+          <mesh>
+            <scale>1 1 1</scale>
+            <uri>model://Light_seeker/meshes/Light_seeker_base_2.dae</uri>
+          </mesh>
+        </geometry>
+      </collission>
       <velocity_decay/>
       <self_collide>0</self_collide>
