Commit message: Tune nav params and update sensor model and RViz
Comment out oakd collision primitive and disable AMCL block. Adjust Nav2
parameters: costmap sizes/resolution/origins, STVL decay and map save
duration, observation ranges/filters, controller timeouts and
thresholds, various stds and limits, and sensor topics. Add a Path
display to seeker.rviz.

File: ros_ws/src/s_description/model/Sensors/oakd/model.sdf.xacro (robot description, xacro)
@@ -23,5 +23,5 @@
           </geometry>
         </visual>
-        <collision name="${base_frame}_collision">
+        <!--<collision name="${base_frame}_collision">
           <pose relative_to="${base_frame}">${collision_offset_x} ${collision_offset_y} ${collision_offset_z} 0 0 0</pose>
           <geometry>
@@ -30,5 +30,5 @@
             </box>
           </geometry>
-        </collision>
+        </collision>-->
         <inertial>
           <mass>${mass}</mass>
